File: pcb/vent_sys/vent_sys.kicad_pcb (KiCad board)
At the start: 2 copper layers, 21 parts, among them J1 Screw_Terminal_01x02, J2 Screw_Terminal_01x02, Q1 BT138-600, U1 PC817, U2 stm32f103c8t6-module-china, U3 MOC3021M, U4 RA-02

Commit message: PCB trace completed
Parts:
- removed R10, R11: 5K, Resistor_SMD:R_1206_3216Metric
- C2: footprint Capacitor_THT:C_Rect_L9.0mm_W9.8mm_P7.50mm_MKT -> Capacitor_THT:C_Rect_L9.0mm_W3.2mm_P7.50mm_MKT
- moved J2 112.5 mm to (65.7, 80.0), turned to 90 degrees
- moved R8 87.3 mm to (71.9, 97.4), turned to 90 degrees
- moved C1 85.8 mm to (67.1, 94.4), turned to 90 degrees
- moved R9 85.4 mm to (89.0, 89.0)
- moved C2 83.0 mm to (84.7, 98.9)
- moved R7 80.5 mm to (63.5, 96.5), turned to 90 degrees
- moved Q1 79.8 mm to (80.3, 94.5)
- moved U3 33.2 mm to (103.0, 92.7), turned to 180 degrees
- moved U4 15.5 mm to (139.2, 75.7)
- moved PS1 15.2 mm to (87.9, 75.7)
- moved R3 14.6 mm to (72.6, 63.0)
- moved J1 12.9 mm to (65.5, 64.8)
- moved R4 12.7 mm to (82.8, 59.4)
- moved R6 12.3 mm to (121.7, 96.8), turned to 270 degrees
- moved R2 5.49 mm to (90.9, 55.4)
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Connections:
- R5 pad 1: Net-(R5-Pad1) -> VCC
- U2 pad 38: Net-(R5-Pad1) -> VCC
- U4 pad 1: Net-(U2-Pad39) -> Net-(U4-Pad1)
- U4 pad 13: Net-(R11-Pad2) -> /MISO
- U4 pad 14: Net-(R10-Pad1) -> /MOSI
- U4 pad 2: Net-(U2-Pad39) -> Net-(U4-Pad2)
- U4 pad 3: Net-(R5-Pad1) -> VCC
- U4 pad 9: Net-(U2-Pad39) -> Net-(U4-Pad9)
Routing:
- net VCC: track 8.49 -> 175.1 mm
- net Net-(R5-Pad1): track 84.0 -> 0.00 mm
- net /L: track 40.7 -> 86.5 mm
- net Net-(R7-Pad1): track 0.00 -> 39.4 mm
- net Net-(C1-Pad2): track 0.00 -> 29.4 mm
- net /MOSI: track 0.00 -> 25.7 mm
- net GND: track 84.3 -> 58.7 mm
- net Net-(R6-Pad2): track 3.14 -> 27.6 mm
- net /MISO: track 0.00 -> 24.0 mm
- net Net-(U2-Pad39): track 11.7 -> 30.8 mm
- net Net-(C1-Pad1): track 0.00 -> 16.2 mm
- net Net-(Q1-Pad3): track 0.00 -> 15.5 mm
- net /SCK: track 34.9 -> 20.8 mm
- net /NSS: track 42.0 -> 29.3 mm
- net /Reset: track 28.7 -> 17.2 mm
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Other:
- board outline added: 88.9 x 53.3 mm
